File: hardware/voltage_indicator.kicad_pcb (KiCad board)
At the start: 2 copper layers, 48 x 62 mm, 60 parts, among them J1 HV+, J2 HV-, Q1 BC807, Q2 TK3P80ERQ, U1 LM211DT, U2 LT8316EFE

Commit message: Update component values
Parts:
- C10: value DNP -> 330u
- R1: value 1k2 -> 1k
- R11: value TBD -> 1k5
- R12: value TBD -> 470R
Changed lines of the file:
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@@
   (net 10 "Net-(R3-Pad1)")
   (net 11 "Net-(R4-Pad1)")
-  (net 12 "Net-(#FLG03-pwr)")
+  (net 12 "Net-(D5-K)")
   (net 13 "Net-(Q1-C)")
   (net 14 "Net-(Q2-G)")
@@
   (net 27 "Net-(R6-Pad1)")
   (net 28 "Net-(R11-Pad1)")
-  (net 29 "Net-(#FLG04-pwr)")
+  (net 29 "Net-(D4-A)")
   (net 30 "Net-(J1-Pin_1)")
   (footprint "Resistor_SMD:R_0603_1608Metric" (layer "F.Cu")
@@
         (effects (font (size 1 1) (thickness 0.15)))
     )
-    (fp_text value "1k2" (at 0 1.43) (layer "F.Fab")
+    (fp_text value "1k" (at 0 1.43) (layer "F.Fab")
         (effects (font (size 1 1) (thickness 0.15)))
     )
@@
       (net 4 "Net-(D3-K)") (pintype "passive"))
     (pad "2" smd roundrect (at 0.775 0) (size 0.9 0.95) (layers "F.Cu" "F.Paste" "F.Mask") (roundrect_rratio 0.25)
-      (net 12 "Net-(#FLG03-pwr)") (pintype "passive"))
+      (net 12 "Net-(D5-K)") (pintype "passive"))
     (model "${KICAD6_3DMODEL_DIR}/Capacitor_SMD.3dshapes/C_0603_1608Metric.wrl"
       (offset (xyz 0 0 0))
@@
       (stroke (width 0.1) (type solid)) (layer "F.Fab"))
     (pad "1" smd rect (at -4.15 0 90) (size 3.2 5) (layers "F.Cu" "F.Paste" "F.Mask")
-      (net 12 "Net-(#FLG03-pwr)") (pinfunction "1") (pintype "passive"))
+      (net 12 "Net-(D5-K)") (pinfunction "1") (pintype "passive"))
     (pad "2" smd rect (at 4.15 0 90) (size 3.2 5) (layers "F.Cu" "F.Paste" "F.Mask")
       (net 3 "+12V") (pinfunction "2") (pintype "passive"))
@@
       (stroke (width 0.1) (type solid)) (layer "F.Fab"))
     (pad "1" smd roundrect (at -0.825 0 180) (size 0.8 0.95) (layers "F.Cu" "F.Paste" "F.Mask") (roundrect_rratio 0.25)
-      (net 12 "Net-(#FLG03-pwr)") (pintype "passive"))
+      (net 12 "Net-(D5-K)") (pintype "passive"))
     (pad "2" smd roundrect (at 0.825 0 180) (size 0.8 0.95) (layers "F.Cu" "F.Paste" "F.Mask") (roundrect_rratio 0.25)
       (net 18 "Net-(U2-FB)") (pintype "passive"))
@@
         (effects (font (size 1 1) (thickness 0.15)))
     )
-    (fp_text value "TBD" (at 0 1.43 90) (layer "F.Fab")
+    (fp_text value "1k5" (at 0 1.43 90) (layer "F.Fab")
         (effects (font (size 1 1) (thickness 0.15)))
     )
@@
       (stroke (width 0.1) (type solid)) (layer "F.Fab"))
     (pad "1" smd rect (at -2.825001 -2.925) (size 1.4612 0.3508) (layers "F.Cu" "F.Paste" "F.Mask")
-      (net 29 "Net-(#FLG04-pwr)") (pinfunction "VIN") (pintype "power_in"))
+      (net 29 "Net-(D4-A)") (pinfunction "VIN") (pintype "power_in"))
     (pad "2" smd rect (at -2.825001 -2.274999) (size 1.4612 0.3508) (layers "F.Cu" "F.Paste" "F.Mask")
-      (net 29 "Net-(#FLG04-pwr)") (pinfunction "VIN") (pintype "power_in"))
+      (net 29 "Net-(D4-A)") (pinfunction "VIN") (pintype "power_in"))
     (pad "3" smd rect (at -2.825001 -1.625001) (size 1.4612 0.3508) (layers "F.Cu" "F.Paste" "F.Mask")
-      (net 29 "Net-(#FLG04-pwr)") (pinfunction "VIN") (pintype "power_in"))
+      (net 29 "Net-(D4-A)") (pinfunction "VIN") (pintype "power_in"))
     (pad "8" smd rect (at -2.825001 1.624998) (size 1.4612 0.3508) (layers "F.Cu" "F.Paste" "F.Mask")
       (net 4 "Net-(D3-K)") (pinfunction "INTVCC") (pintype "passive"))
@@
       (net 5 "Net-(U2-IREG{slash}SS)") (pinfunction "IREG/SS") (pintype "passive"))
     (pad "15" smd rect (at 2.825001 0.325001) (size 1.4612 0.3508) (layers "F.Cu" "F.Paste" "F.Mask")
-      (net 12 "Net-(#FLG03-pwr)") (pinfunction "GND") (pintype "power_in"))
+      (net 12 "Net-(D5-K)") (pinfunction "GND") (pintype "power_in"))
     (pad "16" smd rect (at 2.825001 -0.324998) (size 1.4612 0.3508) (layers "F.Cu" "F.Paste" "F.Mask")
-      (net 12 "Net-(#FLG03-pwr)") (pinfunction "SMODE") (pintype "passive"))
+      (net 12 "Net-(D5-K)") (pinfunction "SMODE") (pintype "passive"))
     (pad "17" smd rect (at 2.825001 -0.974999) (size 1.4612 0.3508) (layers "F.Cu" "F.Paste" "F.Mask")
       (net 4 "Net-(D3-K)") (pinfunction "EN/UVLO") (pintype "passive"))
@@
       (net 14 "Net-(Q2-G)") (pinfunction "GATE") (pintype "output"))
     (pad "20" smd rect (at 2.825001 -2.924998) (size 1.4612 0.3508) (layers "F.Cu" "F.Paste" "F.Mask")
-      (net 12 "Net-(#FLG03-pwr)") (pinfunction "GND") (pintype "power_in"))
+      (net 12 "Net-(D5-K)") (pinfunction "GND") (pintype "power_in"))
     (pad "EPAD" smd rect (at 0.47 0) (size 1.78 5.680001) (layers "F.Cu" "F.Paste" "F.Mask")
-      (net 12 "Net-(#FLG03-pwr)") (pinfunction "EPAD") (pintype "power_in"))
+      (net 12 "Net-(D5-K)") (pinfunction "EPAD") (pintype "power_in"))
   )
   (footprint "Resistor_SMD:R_0603_1608Metric" (layer "F.Cu")
@@
       (net 5 "Net-(U2-IREG{slash}SS)") (pintype "passive"))
     (pad "2" smd roundrect (at 0.775 0) (size 0.9 0.95) (layers "F.Cu" "F.Paste" "F.Mask") (roundrect_rratio 0.25)
-      (net 12 "Net-(#FLG03-pwr)") (pintype "passive"))
+      (net 12 "Net-(D5-K)") (pintype "passive"))
     (model "${KICAD6_3DMODEL_DIR}/Capacitor_SMD.3dshapes/C_0603_1608Metric.wrl"
       (offset (xyz 0 0 0))
@@
         (effects (font (size 1 1) (thickness 0.15)))
     )
-    (fp_text value "TBD" (at 0 1.43) (layer "F.Fab")
+    (fp_text value "470R" (at 0 1.43) (layer "F.Fab")
         (effects (font (size 1 1) (thickness 0.15)))
     )
@@
       (net 1 "VCC") (pinfunction "K") (pintype "passive"))
     (pad "2" smd roundrect (at 0.7 0 180) (size 0.6 0.7) (layers "F.Cu" "F.Paste" "F.Mask") (roundrect_rratio 0.25)
-      (net 29 "Net-(#FLG04-pwr)") (pinfunction "A") (pintype "passive"))
+      (net 29 "Net-(D4-A)") (pinfunction "A") (pintype "passive"))
     (model "${KICAD6_3DMODEL_DIR}/Diode_SMD.3dshapes/D_SOD-523.wrl"
       (offset (xyz 0 0 0))
@@
         (effects (font (size 1 1) (thickness 0.15)))
     )
-    (fp_text value "DNP" (at 0 4.35) (layer "F.Fab")
+    (fp_text value "330u" (at 0 4.35) (layer "F.Fab")
         (effects (font (size 1 1) (thickness 0.15)))
     )
@@
       (stroke (width 0.1) (type solid)) (layer "F.Fab"))
     (pad "1" smd roundrect (at -1.4 0) (size 1.1 1.1) (layers "F.Cu" "F.Paste" "F.Mask") (roundrect_rratio 0.2272727273)
-      (net 12 "Net-(#FLG03-pwr)") (pinfunction "K") (pintype "passive"))
+      (net 12 "Net-(D5-K)") (pinfunction "K") (pintype "passive"))
     (pad "2" smd roundrect (at 1.4 0) (size 1.1 1.1) (layers "F.Cu" "F.Paste" "F.Mask") (roundrect_rratio 0.2272727273)
       (net 2 "GND") (pinfunction "A") (pintype "passive"))
@@
       (net 25 "Net-(C3-Pad1)") (pintype "passive"))
     (pad "2" smd roundrect (at 0.775 0 270) (size 0.9 0.95) (layers "F.Cu" "F.Paste" "F.Mask") (roundrect_rratio 0.25)
-      (net 12 "Net-(#FLG03-pwr)") (pintype "passive"))
+      (net 12 "Net-(D5-K)") (pintype "passive"))
     (model "${KICAD6_3DMODEL_DIR}/Capacitor_SMD.3dshapes/C_0603_1608Metric.wrl"
       (offset (xyz 0 0 0))
@@
       (stroke (width 0.1) (type solid)) (layer "F.Fab"))
     (pad "1" smd roundrect (at -0.825 0 270) (size 0.8 0.95) (layers "F.Cu" "F.Paste" "F.Mask") (roundrect_rratio 0.25)
-      (net 12 "Net-(#FLG03-pwr)") (pintype "passive"))
+      (net 12 "Net-(D5-K)") (pintype "passive"))
     (pad "2" smd roundrect (at 0.825 0 270) (size 0.8 0.95) (layers "F.Cu" "F.Paste" "F.Mask") (roundrect_rratio 0.25)
       (net 24 "Net-(Q2-S)") (pintype "passive"))
@@
       (stroke (width 0.05) (type solid)) (fill none) (layer "B.CrtYd"))
     (pad "1" smd circle (at 0 0 180) (size 1 1) (layers "B.Cu" "B.Mask")
-      (net 12 "Net-(#FLG03-pwr)") (pinfunction "1") (pintype "passive"))
+      (net 12 "Net-(D5-K)") (pinfunction "1") (pintype "passive"))
   )
   (footprint "TestPoint:TestPoint_Pad_D1.0mm" (layer "B.Cu")
@@
       (stroke (width 0.05) (type solid)) (fill none) (layer "B.CrtYd"))
     (pad "1" smd circle (at 0 0 180) (size 1 1) (layers "B.Cu" "B.Mask")
-      (net 29 "Net-(#FLG04-pwr)") (pinfunction "1") (pintype "passive"))
+      (net 29 "Net-(D4-A)") (pinfunction "1") (pintype "passive"))
   )
   (footprint "TestPoint:TestPoint_Pad_D1.0mm" (layer "B.Cu")
@@
     )
   )
-  (zone (net 29) (net_name "Net-(#FLG04-pwr)") (layer "F.Cu") (hatch edge 0.508)
+  (zone (net 29) (net_name "Net-(D4-A)") (layer "F.Cu") (hatch edge 0.508)
     (priority 1)
     (connect_pads yes (clearance 0.508))
@@
     )
   )
-  (zone (net 12) (net_name "Net-(#FLG03-pwr)") (layer "F.Cu") (hatch edge 0.5)
+  (zone (net 12) (net_name "Net-(D5-K)") (layer "F.Cu") (hatch edge 0.5)
     (priority 4)
     (connect_pads yes (clearance 0.1))
@@
     )
   )
-  (zone (net 29) (net_name "Net-(#FLG04-pwr)") (layer "F.Cu") (name "$teardrop_padvia$") (hatch edge 0.5)
+  (zone (net 29) (net_name "Net-(D4-A)") (layer "F.Cu") (name "$teardrop_padvia$") (hatch edge 0.5)
     (priority 30026)
     (attr (teardrop (type padvia)))
@@
     )
   )
-  (zone (net 12) (net_name "Net-(#FLG03-pwr)") (layer "F.Cu") (hatch edge 0.508)
+  (zone (net 12) (net_name "Net-(D5-K)") (layer "F.Cu") (hatch edge 0.508)
     (connect_pads (clearance 0.508))
     (min_thickness 0.254) (filled_areas_thickness no)
@@
     )
   )
-  (zone (net 12) (net_name "Net-(#FLG03-pwr)") (layer "B.Cu") (name "$teardrop_padvia$") (hatch edge 0.5)
+  (zone (net 12) (net_name "Net-(D5-K)") (layer "B.Cu") (name "$teardrop_padvia$") (hatch edge 0.5)
     (priority 30020)
     (attr (teardrop (type padvia)))
@@
     )
   )
-  (zone (net 29) (net_name "Net-(#FLG04-pwr)") (layer "B.Cu") (name "$teardrop_padvia$") (hatch edge 0.5)
+  (zone (net 29) (net_name "Net-(D4-A)") (layer "B.Cu") (name "$teardrop_padvia$") (hatch edge 0.5)
     (priority 30017)
     (attr (teardrop (type padvia)))
